File: 2016/eagle/arduino_mega_shield.sch (EAGLE design)
At the start: 16 parts

Commit message: working on mega shield
Parts:
- removed SDCARD: (no value), SparkFun-Connectors:M07LOCK
- removed U$2: CREATIVE_COMMONS, SparkFun:CREATIVE_COMMONS
- added 3.3V, 5V, GND, I2C2: (no value), SparkFun-Connectors:M04LOCK
- added SPI1, SPI2, SPI3: (no value), SparkFun-Connectors:M06LOCK
Connections:
- removed net CS1: JP3.3, SDCARD.2
- removed net D8: JP3.1
- removed net D9: JP3.2
- new net SS1: JP3.3, SPI1.2
- new net SS2: JP3.2, SPI2.2
- new net SS3: JP3.1, SPI3.2
- net 3.3: now also 3.3V.1, 3.3V.2, 3.3V.3, 3.3V.4; no longer SDCARD.6
- net 5V: now also 5V.1, 5V.2, 5V.3, 5V.4, I2C2.4, SPI1.6, SPI2.6, SPI3.6; no longer SDCARD.7
- net GND: now also GND.1, GND.2, GND.3, GND.4, I2C2.1, SPI1.1, SPI2.1, SPI3.1; no longer SDCARD.1
- net MISO: now also SPI1.4, SPI2.4, SPI3.4; no longer SDCARD.4
- net MOSI: now also SPI1.3, SPI2.3, SPI3.3; no longer SDCARD.3
- net SCK: now also SPI1.5, SPI2.5, SPI3.5; no longer SDCARD.5
- net SCL: now also I2C2.3
- net SDA: now also I2C2.2
