File: 2016/eagle/arduino_mega_shield.brd (EAGLE design)
At the start: 72.4 x 53.3 mm, 16 parts

Commit message: working on mega shield
Parts:
- removed SDCARD: (no value), SparkFun-Connectors:1X07_LOCK
- removed U$2: CREATIVE_COMMONS, SparkFun:CREATIVE_COMMONS
- added 3.3V, 5V, GND, I2C2: (no value), SparkFun-Connectors:1X04_LOCK
- added SPI1, SPI2, SPI3: (no value), SparkFun-Connectors:1X06_LOCK
- moved R3 20.8 mm to (26.7, 24.5), turned to 270 degrees
- moved R1 15.5 mm to (30.5, 24.3), turned to 90 degrees
- moved UART3 8.89 mm to (64.8, 29.2)
- moved LED1 5.08 mm to (27.9, 14.0)
- moved UART2 5.08 mm to (72.4, 29.2)
- moved I2C1 1.80 mm to (80.0, 15.2)
- moved UART1 1.27 mm to (80.0, 29.2)
Connections:
- removed net CS1: JP3.3, SDCARD.2
- removed net D8: JP3.1
- removed net D9: JP3.2
- new net SS1: JP3.3, SPI1.2
- new net SS2: JP3.2, SPI2.2
- new net SS3: JP3.1, SPI3.2
- net 3.3: now also 3.3V.1, 3.3V.2, 3.3V.3, 3.3V.4; no longer SDCARD.6
- net 5V: now also 5V.1, 5V.2, 5V.3, 5V.4, I2C2.4, SPI1.6, SPI2.6, SPI3.6; no longer SDCARD.7
- net GND: now also GND.1, GND.2, GND.3, GND.4, I2C2.1, SPI1.1, SPI2.1, SPI3.1; no longer SDCARD.1
- net MISO: now also SPI1.4, SPI2.4, SPI3.4; no longer SDCARD.4
- net MOSI: now also SPI1.3, SPI2.3, SPI3.3; no longer SDCARD.3
- net SCK: now also SPI1.5, SPI2.5, SPI3.5; no longer SDCARD.5
- net SCL: now also I2C2.3
- net SDA: now also I2C2.2
Routing:
- net GND: track 132.5 -> 0.00 mm
- net 5V: track 110.9 -> 0.00 mm
- net 3.3: track 40.9 -> 0.00 mm
- net SDA: track 32.9 -> 0.00 mm
- net RES: track 31.8 -> 0.00 mm
- net SCL: track 31.2 -> 0.00 mm
- net UART_RX2: track 20.5 -> 0.00 mm
- net UART_RX1: track 20.0 -> 0.00 mm
- net UART_RX3: track 20.0 -> 0.00 mm
- net UART_TX3: track 18.7 -> 0.00 mm
- net UART_TX2: track 18.2 -> 0.00 mm
- net UART_TX1: track 17.6 -> 0.00 mm
- net MOSI: track 11.7 -> 0.00 mm
- net SCK: track 11.7 -> 0.00 mm
- net MISO: track 11.2 -> 0.00 mm
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Other:
- board text added: "3.3V"
- board text added: "Copyright 2016 Grove Enterprises LLC"
- board text added: "I2C1"
- board text added: "I2C2"
- board text added: "Mega Comms Shield 1.0"
- board text added: "SPI1"
- board text added: "SPI2"
- board text added: "SPI3"
- board text added: "UART1"
- board text added: "UART2"
- board text added: "UART3"

Commit message: move labels to correct layer
Parts:
- moved SPI1 4.58 mm to (34.3, 41.9)
- moved SPI2 4.58 mm to (41.9, 41.9)
- moved SPI3 4.58 mm to (49.5, 41.9)
Routing:
- net GND: track 0.00 -> 151.5 mm
- net 5V: track 0.00 -> 115.5 mm
- net SDA: track 0.00 -> 42.4 mm
- net SCL: track 0.00 -> 40.8 mm
- net SCK: track 0.00 -> 36.9 mm
- net RES: track 0.00 -> 34.9 mm
- net MISO: track 0.00 -> 32.7 mm
- net MOSI: track 0.00 -> 31.0 mm
- net 3.3: track 0.00 -> 22.0 mm
- net UART_RX3: track 0.00 -> 21.5 mm
- net UART_RX2: track 0.00 -> 20.4 mm
- net UART_RX1: track 0.00 -> 19.6 mm
- net UART_TX3: track 0.00 -> 18.3 mm
- net UART_TX2: track 0.00 -> 17.3 mm
- net UART_TX1: track 0.00 -> 17.1 mm
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Other:
- board text added: "MISO"
- board text added: "MOSI"
- board text added: "SCK"
- board text added: "SS"
